File: Custom Board/PCB/Custom USB_N64_smaller.brd (EAGLE design)
At the start: 68 x 38.1 mm, 24 parts, among them J1 N64_Data, J2 N64_GND, U1 STM32F446RET6

Commit message: Updated custom board info
Parts:
- added J3: GC_Data, SparkFun-Connectors:1X01
- added J4: GC_GND, SparkFun-Connectors:1X01
- moved C4 21.0 mm to (45.4, 27.9)
- moved C12 20.4 mm to (48.4, 27.9)
- moved J1 9.06 mm to (55.7, 13.9)
- moved J2 9.06 mm to (55.7, 6.24)
- moved U$6 6.89 mm to (35.9, 27.9), turned to 90 degrees
- moved R2 6.40 mm to (23.4, 4.62)
- moved C8 4.35 mm to (50.9, 5.59), turned to 270 degrees
- moved C11 3.89 mm to (29.9, 27.9)
- moved R3 3.76 mm to (26.5, 4.62), turned to 90 degrees
- moved R4 2.82 mm to (29.9, 4.62)
- moved C13 1.95 mm to (32.9, 4.62)
- moved C3 1.41 mm to (33.0, 27.9)
- moved C10 1.39 mm to (42.2, 27.9)
- moved C9 1.00 mm to (47.9, 22.3)
- moved R1 1.00 mm to (14.0, 28.2)
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Connections:
- net GND: now also J4.1
- net N$8: now also J3.1
Routing:
- net 3V3: track 86.2 -> 97.2 mm
- net N$8: track 25.3 -> 35.5 mm
- net N$13: track 9.30 -> 2.96 mm
- net N$5: track 11.8 -> 15.7 mm
- net N$10: track 30.3 -> 33.3 mm
- net +5V: track 60.6 -> 62.6 mm
- net N$12: track 5.08 -> 3.80 mm
- net N$7: track 10.6 -> 9.58 mm
- net DP_USBA: track 14.2 -> 13.2 mm
- net DM_USBA: track 19.3 -> 18.3 mm
- net N$11: track 4.62 -> 3.62 mm
- net DP: track 25.8 -> 25.1 mm
- net N$6: track 4.75 -> 4.16 mm
Other:
- board size 68 x 38.1 mm -> 68 x 36.1 mm
