File: Custom Board/PCB/Custom USB_N64_smaller.sch (EAGLE design)
At the start: 24 parts, among them J1 N64_Data, J2 N64_GND, U1 STM32F446RET6

Commit message: Updated custom board info
Parts:
- added J3: GC_Data, SparkFun-Connectors:M01PTH
- added J4: GC_GND, SparkFun-Connectors:M01PTH
Connections:
- net GND: now also J4.1
- net N$8: now also J3.1
Changed lines of the file:
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@@
 <layers>
 <layer number="1" name="Top" color="4" fill="1" visible="no" active="no"/>
+<layer number="2" name="Route2" color="1" fill="3" visible="no" active="no"/>
+<layer number="3" name="Route3" color="4" fill="3" visible="no" active="no"/>
+<layer number="4" name="Route4" color="1" fill="4" visible="no" active="no"/>
+<layer number="5" name="Route5" color="4" fill="4" visible="no" active="no"/>
+<layer number="6" name="Route6" color="1" fill="8" visible="no" active="no"/>
+<layer number="7" name="Route7" color="4" fill="8" visible="no" active="no"/>
+<layer number="8" name="Route8" color="1" fill="2" visible="no" active="no"/>
+<layer number="9" name="Route9" color="4" fill="2" visible="no" active="no"/>
+<layer number="10" name="Route10" color="1" fill="7" visible="no" active="no"/>
+<layer number="11" name="Route11" color="4" fill="7" visible="no" active="no"/>
+<layer number="12" name="Route12" color="1" fill="5" visible="no" active="no"/>
+<layer number="13" name="Route13" color="4" fill="5" visible="no" active="no"/>
+<layer number="14" name="Route14" color="1" fill="6" visible="no" active="no"/>
+<layer number="15" name="Route15" color="4" fill="6" visible="no" active="no"/>
 <layer number="16" name="Bottom" color="1" fill="1" visible="no" active="no"/>
 <layer number="17" name="Pads" color="2" fill="1" visible="no" active="no"/>
@@
 <part name="GND15" library="supply1" library_urn="urn:adsk.eagle:library:371" deviceset="GND" device=""/>
 <part name="SUPPLY8" library="supply2" library_urn="urn:adsk.eagle:library:372" deviceset="+5V" device=""/>
+<part name="J3" library="SparkFun-Connectors" deviceset="M01" device="PTH" value="GC_Data"/>
+<part name="J4" library="SparkFun-Connectors" deviceset="M01" device="PTH" value="GC_GND"/>
 </parts>
 <sheets>
@@
 <instance part="GND15" gate="1" x="-121.92" y="86.36" rot="R270"/>
 <instance part="SUPPLY8" gate="+5V" x="-160.02" y="2.54" rot="R270"/>
+<instance part="J3" gate="G$1" x="-220.98" y="48.26" rot="R270"/>
+<instance part="J4" gate="G$1" x="-182.88" y="48.26" rot="R270"/>
 </instances>
 <busses>
@@
 <wire x1="-195.58" y1="40.64" x2="-195.58" y2="35.56" width="0.1524" layer="91"/>
 <pinref part="GND11" gate="1" pin="GND"/>
+<pinref part="J4" gate="G$1" pin="1"/>
+<wire x1="-182.88" y1="40.64" x2="-182.88" y2="35.56" width="0.1524" layer="91"/>
+<wire x1="-182.88" y1="35.56" x2="-195.58" y2="35.56" width="0.1524" layer="91"/>
+<junction x="-195.58" y="35.56"/>
 </segment>
 <segment>
@@
 <pinref part="U1" gate="G$1" pin="PA8/MCO1/TIM1_CH1/I2C3_SCL/USART1_CK/OTG_FS_SOF/EVENTOUT"/>
 <wire x1="-132.08" y1="12.7" x2="-208.28" y2="12.7" width="0.1524" layer="91"/>
-<wire x1="-208.28" y1="12.7" x2="-208.28" y2="40.64" width="0.1524" layer="91"/>
-</segment>
-</net>
+<wire x1="-208.28" y1="12.7" x2="-208.28" y2="35.56" width="0.1524" layer="91"/>
+<pinref part="J3" gate="G$1" pin="1"/>
+<wire x1="-208.28" y1="35.56" x2="-208.28" y2="40.64" width="0.1524" layer="91"/>
+<wire x1="-220.98" y1="40.64" x2="-220.98" y2="35.56" width="0.1524" layer="91"/>
+<wire x1="-220.98" y1="35.56" x2="-208.28" y2="35.56" width="0.1524" layer="91"/>
+<junction x="-208.28" y="35.56"/>
+</segment>
+</net>
